Commit message: Fix slipping & precision loss in gazebo model

File: catkin_ws/src/kt_gazebo/src/kt_gazebo.xacro (robot description, xacro)
@@ -5,6 +5,7 @@
   <!-- Import Rviz colors -->
   <xacro:include filename="$(find kt_gazebo)/src/materials.xacro" />
-  <xacro:property name="INF" value="1.0e+100"/>
+  <xacro:property name="INF" value="1.0e+50"/>
   <xacro:property name="PI" value="3.1415926535897931"/>
+  <xacro:property name="MAX_RPS" value="3.2724895833333334"/>
   <xacro:macro name="servo" params="suffix">
     <link name="servo_${suffix}">
@@ -26,9 +27,10 @@
     </link>
   </xacro:macro>
-  <xacro:macro name="wheel" params="suffix">
+  <xacro:macro name="wheel" params="suffix reflect">
     <link name='wheel_${suffix}'>
       <inertial>
         <mass value="0.03"/>
-        <inertia ixx="8.48e-06" ixy="0" ixz="0" iyy="8.48e-06" iyz="0" izz="1.584e-05"/>
+        <!-- We multiply the inertial values by 100x to prevent slippage/loss of precision by ODE. -->
+        <inertia ixx="8.48e-04" ixy="0" ixz="0" iyy="8.48e-04" iyz="0" izz="1.584e-03"/>
       </inertial>
       <visual name='visual'>
@@ -44,4 +46,12 @@
       </collision>
     </link>
+    <joint name='wheel_${suffix}_joint' type='revolute'>
+      <origin xyz="${reflect*0.087537} 0.04 -0.013883" rpy="0 ${PI/2} 0"/>
+      <parent link="base"/>
+      <child link="wheel_${suffix}"/>
+      <limit effort="7" velocity="${MAX_RPS}" lower="-${INF}" upper="${INF}"/>
+      <axis xyz="0 0 -1"/>
+      <dynamics damping="1.0" friction="0.00"/>
+    </joint>
   </xacro:macro>
   <!-- <origin xyz="0.000537 0.007761 0.214993" rpy="0 0 0"/> -->
@@ -82,31 +92,15 @@
   </xacro:servo>
   <joint name='servo_l_fix' type='fixed'>
-    <origin xyz="-0.056463 0.041761 -0.013883" rpy="0 0 -${PI}" />
+    <origin xyz="-0.057537 0.03 -0.013883" rpy="0 0 -${PI}" />
     <parent link="base"/>
     <child link="servo_left"/>
   </joint>
   <joint name='servo_r_fix' type='fixed'>
-    <origin xyz="0.057537 0.041761 -0.013883" rpy="0 0 0" />
+    <origin xyz="0.057537 0.03 -0.013883" rpy="0 0 0" />
     <parent link="base"/>
     <child link="servo_right"/>
   </joint>
-  <xacro:wheel suffix='left'/>
-  <joint name='wheel_left_rev' type='revolute'>
-    <origin xyz="-0.086463 0.051761 -0.013883" rpy="0 ${PI/2} 0"/>
-    <parent link="base"/>
-    <child link="wheel_left"/>
-    <limit effort="0.1" velocity="1.0" lower="-${INF}" upper="${INF}"/>
-    <axis xyz="0 0 -1"/>
-    <dynamics damping="0.001" friction="0.01"/>
-  </joint>
-  <xacro:wheel suffix='right'/>
-  <joint name='wheel_right_rev' type='revolute'>
-    <origin xyz="0.087537 0.051761 -0.013883" rpy="0 ${PI/2} 0"/>
-    <parent link="base"/>
-    <child link="wheel_right"/>
-    <limit effort="0.1" velocity="1.0" lower="-${INF}" upper="${INF}"/>
-    <axis xyz="0 0 -1"/>
-    <dynamics damping="0.001" friction="0.01"/>
-  </joint>
+  <xacro:wheel suffix='left' reflect="1"/>
+  <xacro:wheel suffix='right' reflect="-1"/>
   <link name='back_stack'>
     <inertial>
@@ -127,5 +121,5 @@
   </link>
   <joint name='back_stack_f' type='fixed'>
-    <origin xyz="0.000271 -0.039485 -0.019055" rpy="0 0 0"/>
+    <origin xyz="0 -0.05 -0.02" rpy="0 0 0"/>
     <parent link="base"/>
     <child link="back_stack"/>
@@ -148,14 +142,12 @@
     </collision>
   </link>
-  <joint name='lidar_rev' type='revolute'>
-    <origin xyz="0.000271 0.036043 0.063556" rpy="0 0 0"/>
+  <joint name='lidar_top' type='fixed'>
+    <origin xyz="0 0.02 0.06" rpy="0 0 0"/>
     <parent link="base"/>
     <child link="lidar"/>
-    <limit effort="0.1" velocity="1.0" lower="-${INF}" upper="${INF}"/>
-    <axis xyz="0 0 1"/>
   </joint>
   <transmission name="tran1">
     <type>transmission_interface/SimpleTransmission</type>
-    <joint name="wheel_left_rev">
+    <joint name="wheel_left_joint">
       <hardwareInterface>hardware_interface/EffortJointInterface</hardwareInterface>
     </joint>
@@ -167,5 +159,5 @@
   <transmission name="tran2">
     <type>transmission_interface/SimpleTransmission</type>
-    <joint name="wheel_right_rev">
+    <joint name="wheel_right_joint">
       <hardwareInterface>hardware_interface/EffortJointInterface</hardwareInterface>
     </joint>

Commit message: Added differential drive via gui

File: catkin_ws/src/kt_gazebo/src/kt_gazebo.xacro (robot description, xacro)
@@ -46,12 +46,21 @@
       </collision>
     </link>
-    <joint name='wheel_${suffix}_joint' type='revolute'>
+    <joint name='wheel_${suffix}_joint' type='continuous'>
       <origin xyz="${reflect*0.087537} 0.04 -0.013883" rpy="0 ${PI/2} 0"/>
       <parent link="base"/>
       <child link="wheel_${suffix}"/>
-      <limit effort="7" velocity="${MAX_RPS}" lower="-${INF}" upper="${INF}"/>
+      <limit effort="7" velocity="${MAX_RPS}"/>
       <axis xyz="0 0 -1"/>
       <dynamics damping="1.0" friction="0.00"/>
     </joint>
+    <transmission name="wheel_${suffix}_trans">
+      <type>transmission_interface/SimpleTransmission</type>
+      <joint name="wheel_${suffix}_joint">
+        <hardwareInterface>hardware_interface/VelocityJointInterface</hardwareInterface>
+      </joint>
+      <actuator name="wheel_${suffix}_motor">
+        <mechanicalReduction>1</mechanicalReduction>
+      </actuator>
+    </transmission>
   </xacro:macro>
   <!-- <origin xyz="0.000537 0.007761 0.214993" rpy="0 0 0"/> -->
@@ -101,6 +110,6 @@
     <child link="servo_right"/>
   </joint>
-  <xacro:wheel suffix='left' reflect="1"/>
-  <xacro:wheel suffix='right' reflect="-1"/>
+  <xacro:wheel suffix='left' reflect="-1"/>
+  <xacro:wheel suffix='right' reflect="1"/>
   <link name='back_stack'>
     <inertial>
@@ -147,23 +156,3 @@
     <child link="lidar"/>
   </joint>
-  <transmission name="tran1">
-    <type>transmission_interface/SimpleTransmission</type>
-    <joint name="wheel_left_joint">
-      <hardwareInterface>hardware_interface/EffortJointInterface</hardwareInterface>
-    </joint>
-    <actuator name="motor1">
-      <hardwareInterface>hardware_interface/EffortJointInterface</hardwareInterface>
-      <mechanicalReduction>1</mechanicalReduction>
-    </actuator>
-  </transmission>
-  <transmission name="tran2">
-    <type>transmission_interface/SimpleTransmission</type>
-    <joint name="wheel_right_joint">
-      <hardwareInterface>hardware_interface/EffortJointInterface</hardwareInterface>
-    </joint>
-    <actuator name="motor2">
-      <hardwareInterface>hardware_interface/EffortJointInterface</hardwareInterface>
-      <mechanicalReduction>1</mechanicalReduction>
-    </actuator>
-  </transmission>
 </robot>

Commit message: Switched ktbot xacro file to be x-forward to match sim odometry

File: catkin_ws/src/kt_gazebo/src/kt_gazebo.xacro (robot description, xacro)
@@ -12,9 +12,9 @@
       <inertial>
         <mass value="0.052"/>
-        <inertia ixx="1.188e-05" ixy="0" ixz="0" iyy="8.02e-06" iyz="0" izz="1.448e-05"/>
+        <inertia ixx="8.02e-06" ixy="0" ixz="0" iyy="1.188e-05" iyz="0" izz="1.448e-05"/>
       </inertial>
       <visual name='visual'>
         <geometry>
-          <box size="0.035 0.046 0.025"/>
+          <box size="0.046 0.035 0.025"/>
         </geometry>
         <material name="dgrey"/>
@@ -22,5 +22,5 @@
       <collision name='collision'>
         <geometry>
-          <box size="0.035 0.046 0.025"/>
+          <box size="0.046 0.035 0.025"/>
         </geometry>
       </collision>
@@ -30,5 +30,6 @@
     <link name='wheel_${suffix}'>
       <inertial>
-        <mass value="0.03"/>
+        <!-- actual mass is ~0.03 -->
+        <mass value="0.30"/>
         <!-- We multiply the inertial values by 100x to prevent slippage/loss of precision by ODE. -->
         <inertia ixx="8.48e-04" ixy="0" ixz="0" iyy="8.48e-04" iyz="0" izz="1.584e-03"/>
@@ -47,6 +48,6 @@
     </link>
     <joint name='wheel_${suffix}_joint' type='continuous'>
-      <origin xyz="${reflect*0.087537} 0.04 -0.013883" rpy="0 ${PI/2} 0"/>
-      <parent link="base"/>
+      <origin xyz="0.04 ${reflect*0.087537} -0.013883" rpy="${PI/2} ${PI/2} 0"/>
+      <parent link="base_link"/>
       <child link="wheel_${suffix}"/>
       <limit effort="7" velocity="${MAX_RPS}"/>
@@ -65,12 +66,12 @@
   </xacro:macro>
   <!-- <origin xyz="0.000537 0.007761 0.214993" rpy="0 0 0"/> -->
-  <link name='base'>
+  <link name='base_link'>
     <inertial>
       <mass value="0.41"/>
-      <inertia ixx="0.00062306"  ixy="0" ixz="0" iyy="0.00076912" iyz="0" izz="0.00139144"/>
+      <inertia ixx="0.00076912" ixy="0" ixz="0" iyy="0.00062306" iyz="0" izz="0.00139144"/>
     </inertial>
     <visual name='visual'>
       <geometry>
-        <box size="0.15 0.135 0.0033"/>
+        <box size="0.135 0.15 0.0033"/>
       </geometry>
       <material name="white"/>
@@ -79,9 +80,9 @@
     <collision name='collision'>
       <geometry>
-        <box size="0.15 0.135 0.0033"/>
+        <box size="0.135 0.15 0.0033"/>
       </geometry>
     </collision>
     <visual name='caster_visual'>
-      <origin xyz="0.0 -0.05 -0.038" rpy="0 0 0"/>
+      <origin xyz="-0.05 0.0 -0.038" rpy="0 0 0"/>
       <geometry>
         <sphere radius="0.01"/>
@@ -90,5 +91,5 @@
     </visual>
     <collision name='caster_collision'>
-      <origin xyz="0.0 -0.05 -0.038" rpy="0 0 0"/>
+      <origin xyz="-0.05 0.0 -0.038" rpy="0 0 0"/>
       <geometry>
         <sphere radius="0.01"/>
@@ -101,23 +102,23 @@
   </xacro:servo>
   <joint name='servo_l_fix' type='fixed'>
-    <origin xyz="-0.057537 0.03 -0.013883" rpy="0 0 -${PI}" />
-    <parent link="base"/>
+    <origin xyz="0.03 -0.057537 -0.013883" rpy="0 -${PI} 0"/>
+    <parent link="base_link"/>
     <child link="servo_left"/>
   </joint>
   <joint name='servo_r_fix' type='fixed'>
-    <origin xyz="0.057537 0.03 -0.013883" rpy="0 0 0" />
-    <parent link="base"/>
+    <origin xyz="0.03 0.057537 -0.013883" rpy="0 0 0"/>
+    <parent link="base_link"/>
     <child link="servo_right"/>
   </joint>
-  <xacro:wheel suffix='left' reflect="-1"/>
-  <xacro:wheel suffix='right' reflect="1"/>
+  <xacro:wheel suffix='left' reflect="1"/>
+  <xacro:wheel suffix='right' reflect="-1"/>
   <link name='back_stack'>
     <inertial>
       <mass value="0.01"/>
-      <inertia ixx="1.98e-06" ixy="0" ixz="0" iyy="2.3e-06" iyz="0" izz="2.35e-06"/>
+      <inertia ixx="2.3e-06" ixy="0" ixz="0" iyy="1.98e-06" iyz="0" izz="2.35e-06"/>
     </inertial>
     <visual name='visual'>
       <geometry>
-        <box size="0.04 0.035 0.034"/>
+        <box size="0.035 0.04 0.034"/>
       </geometry>
       <material name="white"/>
@@ -125,11 +126,11 @@
     <collision name='collision'>
       <geometry>
-        <box size="0.04 0.035 0.034"/>
+        <box size="0.035 0.04 0.034"/>
       </geometry>
     </collision>
   </link>
   <joint name='back_stack_f' type='fixed'>
-    <origin xyz="0 -0.05 -0.02" rpy="0 0 0"/>
-    <parent link="base"/>
+    <origin xyz="-0.05 0 -0.02" rpy="0 0 0"/>
+    <parent link="base_link"/>
     <child link="back_stack"/>
   </joint>
@@ -152,6 +153,6 @@
   </link>
   <joint name='lidar_top' type='fixed'>
-    <origin xyz="0 0.02 0.06" rpy="0 0 0"/>
-    <parent link="base"/>
+    <origin xyz="0.02 0 0.06" rpy="0 0 0"/>
+    <parent link="base_link"/>
     <child link="lidar"/>
   </joint>
