Commit message: Fix ktbot xacro file to use new bot size

File: catkin_ws/src/ktbot_description/urdf/ktbot.xacro (robot description, xacro)
@@ -48,5 +48,5 @@
     </link>
     <joint name='wheel_${suffix}_joint' type='continuous'>
-      <origin xyz="0.04 ${reflect*0.087537} -0.013883" rpy="${PI/2} ${PI/2} 0"/>
+      <origin xyz="0.0725 ${reflect*0.137537} -0.013883" rpy="${PI/2} ${PI/2} 0"/>
       <parent link="base_link"/>
       <child link="wheel_${suffix}"/>
@@ -73,5 +73,5 @@
     <visual name='visual'>
       <geometry>
-        <box size="0.135 0.15 0.0033"/>
+        <box size="0.2 0.25 0.0033"/>
       </geometry>
       <material name="white"/>
@@ -80,9 +80,10 @@
     <collision name='collision'>
       <geometry>
-        <box size="0.135 0.15 0.0033"/>
+        <!-- <box size="0.135 0.15 0.0033"/> -->
+        <box size="0.2 0.25 0.0033"/>
       </geometry>
     </collision>
     <visual name='caster_visual'>
-      <origin xyz="-0.05 0.0 -0.038" rpy="0 0 0"/>
+      <origin xyz="-0.0825 0.0 -0.038" rpy="0 0 0"/>
       <geometry>
         <sphere radius="0.01"/>
@@ -91,5 +92,5 @@
     </visual>
     <collision name='caster_collision'>
-      <origin xyz="-0.05 0.0 -0.038" rpy="0 0 0"/>
+      <origin xyz="-0.0825 0.0 -0.038" rpy="0 0 0"/>
       <geometry>
         <sphere radius="0.01"/>
@@ -102,10 +103,10 @@
   </xacro:servo>
   <joint name='servo_l_fix' type='fixed'>
-    <origin xyz="0.03 -0.057537 -0.013883" rpy="0 -${PI} 0"/>
+    <origin xyz="0.0625 -0.107537 -0.013883" rpy="0 -${PI} 0"/>
     <parent link="base_link"/>
     <child link="servo_left"/>
   </joint>
   <joint name='servo_r_fix' type='fixed'>
-    <origin xyz="0.03 0.057537 -0.013883" rpy="0 0 0"/>
+    <origin xyz="0.0625 0.107537 -0.013883" rpy="0 0 0"/>
     <parent link="base_link"/>
     <child link="servo_right"/>
@@ -131,5 +132,5 @@
   </link>
   <joint name='back_stack_f' type='fixed'>
-    <origin xyz="-0.05 0 -0.02" rpy="0 0 0"/>
+    <origin xyz="-0.0825 0 -0.02" rpy="0 0 0"/>
     <parent link="base_link"/>
     <child link="back_stack"/>
@@ -153,5 +154,5 @@
   </link>
   <joint name='lidar_top' type='fixed'>
-    <origin xyz="0.02 0 0.06" rpy="0 0 0"/>
+    <origin xyz="0.0525 0 0.06" rpy="0 0 0"/>
     <parent link="base_link"/>
     <child link="lidar"/>

Commit message: added baudrate to serial.cpp

File: catkin_ws/src/ktbot_description/urdf/ktbot.xacro (robot description, xacro)
@@ -136,5 +136,5 @@
     <child link="back_stack"/>
   </joint>
-  <link name='lidar'>
+  <link name='base_laser_link'>
     <inertial>
       <mass value="0.1"/>
@@ -156,5 +156,5 @@
     <origin xyz="0.0525 0 0.06" rpy="0 0 0"/>
     <parent link="base_link"/>
-    <child link="lidar"/>
+    <child link="base_laser_link"/>
   </joint>
 </robot>
