Commit message: Fix inertials on inserter, setup gazebo mimic plugin workaround to lack of support for joint mimicry, refactor launch file and add PID to joints

File: catkin_ws/src/inserter_detector/simulation/inserter/inserter.xacro (robot description, xacro)
@@ -13,14 +13,13 @@
   <xacro:property name="thick" value="0.025" />
   <xacro:property name="l1" value="0.1" />
-  <xacro:property name="servo_inertial">
+  <xacro:macro name="box_inertial" params="x y z mass *origin">
     <inertial>
-      <origin xyz="0 0 ${base_height/2}" rpy="0 0 0"/>
-      <mass value="${mass}"/>
-      <inertia
-        ixx="${mass / 12.0 * (base_width*base_width + base_height*base_height)}" ixy="0.0" ixz="0.0"
-        iyy="${mass / 12.0 * (base_height*base_height + base_width*base_width)}" iyz="0.0"
-        izz="${mass / 12.0 * (base_width*base_width + base_width*base_width)}"/>
+      <mass value="${mass}" />
+      <xacro:insert_block name="origin" />
+      <inertia ixx="${0.0833333 * mass * (y*y + z*z)}" ixy="0.0" ixz="0.0"
+        iyy="${0.0833333 * mass * (x*x + z*z)}" iyz="0.0"
+        izz="${0.0833333 * mass * (x*x + y*y)}" />
     </inertial>
-  </xacro:property>
+  </xacro:macro>
   <!-- Import all Gazebo-customization elements, including Gazebo colors -->
   <xacro:include filename="$(find inserter_detector)/simulation/inserter/inserter.gazebo" />
@@ -48,5 +47,7 @@
       <material name="grey"/>
     </visual>
-    <xacro:insert_block name="servo_inertial"/>
+    <xacro:box_inertial mass="1.0" x="${base_width}" y="${base_width}" z="${base_height}">
+      <origin xyz="0 0 ${base_height/2}" />
+    </xacro:box_inertial>
   </link>
   <joint name="joint1" type="revolute">
@@ -66,4 +67,7 @@
       <material name="dgrey"/>
     </visual>
+    <xacro:box_inertial mass="1.0" x="0.1" y="0.1" z="0.1">
+      <origin xyz="0 0 0" />
+    </xacro:box_inertial>
   </link>
   <joint name="joint2" type="revolute">
@@ -83,4 +87,7 @@
       <material name="dgrey"/>
     </visual>
+    <xacro:box_inertial mass="1.0" x="${thick}" y="${thick}" z="${l1}">
+      <origin xyz="0 0 ${l1/2}" />
+    </xacro:box_inertial>
   </link>
   <joint name="joint3" type="revolute">
@@ -100,4 +107,7 @@
       <material name="dgrey"/>
     </visual>
+    <xacro:box_inertial mass="1.0" x="${thick}" y="${thick}" z="${l1}">
+      <origin xyz="0 0 ${l1/2}" />
+    </xacro:box_inertial>
   </link>
   <joint name="joint4" type="revolute">
@@ -117,4 +127,7 @@
       <material name="dgrey"/>
     </visual>
+    <xacro:box_inertial mass="0.1" x="${thick/2}" y="${l1}" z="${thick/2}">
+      <origin xyz="0 0 0" />
+    </xacro:box_inertial>
   </link>
   <joint name="joint5" type="prismatic">
@@ -133,4 +146,7 @@
       <material name="dgrey"/>
     </visual>
+    <xacro:box_inertial mass="0.1" x="${l1/2}" y="${thick/2}" z="${thick/2}">
+      <origin xyz="${-l1/4} 0 0" />
+    </xacro:box_inertial>
   </link>
   <joint name="joint6" type="prismatic">
@@ -150,14 +166,64 @@
       <material name="dgrey"/>
     </visual>
+    <xacro:box_inertial mass="0.1" x="${l1/2}" y="${thick/2}" z="${thick/2}">
+      <origin xyz="${-l1/4} 0 0" />
+    </xacro:box_inertial>
   </link>
   <transmission name="tran1">
     <type>transmission_interface/SimpleTransmission</type>
-    <joint name="joint1">
-      <hardwareInterface>hardware_interface/EffortJointInterface</hardwareInterface>
-    </joint>
     <actuator name="motor1">
-      <hardwareInterface>hardware_interface/EffortJointInterface</hardwareInterface>
       <mechanicalReduction>1</mechanicalReduction>
     </actuator>
+    <joint name="joint1">
+      <hardwareInterface>hardware_interface/PositionJointInterface</hardwareInterface>
+    </joint>
   </transmission>
+  <transmission name="tran2">
+    <type>transmission_interface/SimpleTransmission</type>
+    <actuator name="motor2">
+      <mechanicalReduction>1</mechanicalReduction>
+    </actuator>
+    <joint name="joint2">
+      <hardwareInterface>hardware_interface/PositionJointInterface</hardwareInterface>
+    </joint>
+  </transmission>
+  <transmission name="tran5">
+    <type>transmission_interface/SimpleTransmission</type>
+    <actuator name="motor5">
+      <mechanicalReduction>1</mechanicalReduction>
+    </actuator>
+    <joint name="joint5">
+      <hardwareInterface>hardware_interface/PositionJointInterface</hardwareInterface>
+    </joint>
+  </transmission>
+  <xacro:macro name="mimic_joint_plugin_gazebo" params="name_prefix parent_joint mimic_joint has_pid:=false multiplier:=1.0 offset:=0 sensitiveness:=0.0 max_effort:=1.0 robot_namespace:=''">
+    <gazebo>
+      <plugin name="${name_prefix}mimic_joint_plugin" filename="libroboticsgroup_gazebo_mimic_joint_plugin.so">
+        <joint>${parent_joint}</joint>
+        <mimicJoint>${mimic_joint}</mimicJoint>
+        <xacro:if value="${has_pid}">                     <!-- if set to true, PID parameters from "/gazebo_ros_control/pid_gains/${mimic_joint}" are loaded -->
+          <hasPID />
+        </xacro:if>
+        <multiplier>${multiplier}</multiplier>
+        <offset>${offset}</offset>
+        <sensitiveness>${sensitiveness}</sensitiveness>   <!-- if absolute difference between setpoint and process value is below this threshold, do nothing; 0.0 = disable [rad] -->
+        <maxEffort>${max_effort}</maxEffort>              <!-- only taken into account if has_pid:=true [Nm] -->
+        <xacro:unless value="${robot_namespace == ''}">
+          <robotNamespace>${robot_namespace}</robotNamespace>
+        </xacro:unless>
+      </plugin>
+    </gazebo>
+  </xacro:macro>
+  <xacro:mimic_joint_plugin_gazebo name_prefix="joint3"
+    parent_joint="joint2" mimic_joint="joint3"
+    has_pid="true" multiplier="-2.0" offset="${PI}" max_effort="20.0"
+    robot_namespace="/inserter"/>
+  <xacro:mimic_joint_plugin_gazebo name_prefix="joint4"
+    parent_joint="joint2" mimic_joint="joint4"
+    has_pid="true" multiplier="1.0" max_effort="20.0"
+    robot_namespace="/inserter"/>
+  <xacro:mimic_joint_plugin_gazebo name_prefix="joint6"
+    parent_joint="joint5" mimic_joint="joint6"
+    has_pid="true" multiplier="1.0" max_effort="100.0"
+    robot_namespace="/inserter"/>
 </robot>

Commit message: Beginning to work on motion planning

File: catkin_ws/src/inserter_detector/simulation/inserter/inserter.xacro (robot description, xacro)
@@ -72,5 +72,5 @@
   </link>
   <joint name="joint2" type="revolute">
-    <limit effort="1000.0" lower="0.1" upper="1.1" velocity="0.5"/>
+    <limit effort="1000.0" lower="0.05" upper="1.1" velocity="0.5"/>
     <origin rpy="0 0 0" xyz="0 0 0"/>
     <parent link="link1"/>
@@ -92,5 +92,5 @@
   </link>
   <joint name="joint3" type="revolute">
-    <limit effort="1000.0" lower="-${PI*0.6}" upper="${PI*0.6}" velocity="0.5"/>
+    <limit effort="1000.0" lower="-${PI}" upper="${PI}" velocity="0.5"/>
     <origin rpy="0 0 0" xyz="0 0 ${l1}"/>
     <parent link="link2"/>
