Commit message: Optimistic commit - halfway through refactoring inserter arm, so it is compatible with moveit software

File: catkin_ws/src/inserter_detector/simulation/inserter/inserter2.xacro (robot description, xacro)
@@ -22,6 +22,14 @@
     </inertial>
   </xacro:macro>
-  <!-- Import all Gazebo-customization elements, including Gazebo colors -->
-  <xacro:include filename="$(find inserter_detector)/simulation/inserter/inserter.gazebo" />
+  <!-- ros_control plugin -->
+  <gazebo>
+    <plugin name="gazebo_ros_control" filename="libgazebo_ros_control.so">
+      <!-- <robotNamespace>$(arg robot_name)</robotNamespace> -->
+      <robotSimType>gazebo_ros_control/DefaultRobotHWSim</robotSimType>
+    </plugin>
+  </gazebo>
+  <gazebo reference="base_link">
+    <material>Gazebo/Black</material>
+  </gazebo>
   <!-- Import Rviz colors -->
   <xacro:include filename="$(find inserter_detector)/simulation/inserter/materials.xacro" />
@@ -34,10 +42,4 @@
   <!-- Base Link -->
   <link name="base_link">
-    <collision>
-      <origin xyz="0 0 ${base_height/2}" rpy="0 0 0"/>
-      <geometry>
-        <box size="${base_width} ${base_width} ${base_height}"/>
-      </geometry>
-    </collision>
     <visual>
       <origin xyz="0 0 ${base_height/2}" rpy="0 0 0"/>
@@ -52,23 +54,23 @@
   </link>
   <joint name="joint1" type="revolute">
-    <limit effort="1000.0" lower="${-PI}" upper="${PI}" velocity="0.5"/>
-    <origin rpy="0 0 0" xyz="0 0 ${base_height + 0.01}"/>
+    <limit effort="1000.0" lower="${-PI/2}" upper="${PI/2}" velocity="5"/>
+    <origin rpy="0 0 0" xyz="0 0 0"/> <!-- ${base_height + 0.01} -->
     <parent link="base_link"/>
     <child link="link1"/>
     <axis xyz="0 0 1"/>
-    <dynamics damping="0.7"/>
+    <dynamics damping="0.4"/>
   </joint>
   <link name="link1">
-    <xacro:box_inertial mass="1.0" x="0.1" y="0.1" z="0.1">
+    <xacro:box_inertial mass="10" x="0.5" y="0.5" z="0.5">
       <origin xyz="0 0 0" />
     </xacro:box_inertial>
   </link>
   <joint name="joint2" type="revolute">
-    <limit effort="1000.0" lower="0.05" upper="1.1" velocity="0.5"/>
-    <origin rpy="0 0 0" xyz="0 0 0"/>
+    <limit effort="1000.0" lower="0.05" upper="1.1" velocity="5"/>
+    <origin rpy="0 0 0" xyz="0 0 ${base_height + 0.01}"/>
     <parent link="link1"/>
     <child link="link2"/>
     <axis xyz="0 1 0"/>
-    <dynamics damping="0.7"/>
+    <dynamics damping="0.4"/>
   </joint>
   <link name="link2">
@@ -80,14 +82,15 @@
       <material name="dgrey"/>
     </visual>
-    <xacro:box_inertial mass="1.0" x="${thick}" y="${thick}" z="${l1}">
+    <xacro:box_inertial mass="0.1" x="${thick}" y="${thick}" z="${l1}">
       <origin xyz="0 0 ${l1/2}" />
     </xacro:box_inertial>
   </link>
   <joint name="joint3" type="revolute">
-    <limit effort="1000.0" lower="0" upper="${PI}" velocity="0.5"/>
+    <limit effort="1000.0" lower="0" upper="${PI}" velocity="5"/>
     <origin rpy="0 0 0" xyz="0 0 ${l1}"/>
     <parent link="link2"/>
     <child link="link3"/>
     <axis xyz="0 1 0"/>
+    <dynamics damping="0.2"/>
   </joint>
   <link name="link3">
@@ -99,20 +102,13 @@
       <material name="dgrey"/>
     </visual>
-    <xacro:box_inertial mass="1.0" x="${thick}" y="${thick}" z="${l1}">
+    <xacro:box_inertial mass="0.1" x="${thick}" y="${thick}" z="${l1}">
       <origin xyz="0 0 ${l1/2}" />
     </xacro:box_inertial>
   </link>
-  <joint name="joint_arm_end" type="fixed">
-    <origin rpy="0 0 0" xyz="0 0 ${l1}"/>
+  <joint name="joint4" type="fixed">
+    <!-- <limit effort="1000.0" lower="-${PI*0.6}" upper="${PI*0.6}" velocity="5"/> -->
+    <origin rpy="0 ${PI/2} 0" xyz="0 0 ${l1}"/>
     <parent link="link3"/>
-    <child link="link_arm_end"/>
-  </joint>
-  <link name="link_arm_end"></link>
-  <joint name="joint4" type="revolute">
-    <limit effort="1000.0" lower="-${PI*0.6}" upper="${PI*0.6}" velocity="0.5"/>
-    <origin rpy="0 0 0" xyz="0 0 0"/>
-    <parent link="link_arm_end"/>
     <child link="link4"/>
-    <mimic joint="joint2" multiplier="1" offset="0"/>
     <axis xyz="0 1 0"/>
   </joint>
@@ -130,9 +126,10 @@
   </link>
   <joint name="joint5" type="prismatic">
-    <limit effort="1000.0" lower="0.01" upper="0.05" velocity="0.5"/>
+    <limit effort="1000.0" lower="0.01" upper="0.05" velocity="5"/>
     <origin rpy="0 0 0" xyz="0 0 0"/>
     <parent link="link4"/>
     <child link="link5"/>
     <axis xyz="0 1 0"/>
+    <dynamics damping="0.2"/>
   </joint>
   <link name="link5">
@@ -147,12 +144,18 @@
       <origin xyz="${-l1/4} 0 0" />
     </xacro:box_inertial>
+    <collision>
+      <origin xyz="${-l1/4} 0 0" rpy="0 0 0"/>
+      <geometry>
+        <box size="${l1/2} ${thick/2} ${thick/2}"/>
+      </geometry>
+    </collision>
   </link>
   <joint name="joint6" type="prismatic">
-    <limit effort="1000.0" lower="0.01" upper="0.05" velocity="0.5"/>
+    <limit effort="1000.0" lower="0.01" upper="0.05" velocity="5"/>
     <origin rpy="0 0 0" xyz="0 0 0"/>
     <parent link="link4"/>
     <child link="link6"/>
     <axis xyz="0 -1 0"/>
-    <mimic joint="joint5" multiplier="1" offset="0"/>
+    <dynamics damping="0.2"/>
   </joint>
   <link name="link6">
@@ -167,4 +170,19 @@
       <origin xyz="${-l1/4} 0 0" />
     </xacro:box_inertial>
+    <collision>
+      <origin xyz="${-l1/4} 0 0" rpy="0 0 0"/>
+      <geometry>
+        <box size="${l1/2} ${thick/2} ${thick/2}"/>
+      </geometry>
+      <surface>
+        <friction>
+          <!-- rubber on rubber, https://www.engineeringtoolbox.com/friction-coefficients-d_778.html -->
+          <ode>
+            <mu>1.16</mu>
+            <mu2>1.16</mu2>
+          </ode>
+        </friction>
+      </surface>
+    </collision>
   </link>
   <transmission name="tran1">
@@ -174,5 +192,5 @@
     </actuator>
     <joint name="joint1">
-      <hardwareInterface>hardware_interface/PositionJointInterface</hardwareInterface>
+      <hardwareInterface>hardware_interface/EffortJointInterface</hardwareInterface>
     </joint>
   </transmission>
@@ -183,5 +201,14 @@
     </actuator>
     <joint name="joint2">
-      <hardwareInterface>hardware_interface/PositionJointInterface</hardwareInterface>
+      <hardwareInterface>hardware_interface/EffortJointInterface</hardwareInterface>
+    </joint>
+  </transmission>
+  <transmission name="tran3">
+    <type>transmission_interface/SimpleTransmission</type>
+    <actuator name="motor3">
+      <mechanicalReduction>1</mechanicalReduction>
+    </actuator>
+    <joint name="joint3">
+      <hardwareInterface>hardware_interface/EffortJointInterface</hardwareInterface>
     </joint>
   </transmission>
@@ -192,32 +219,15 @@
     </actuator>
     <joint name="joint5">
-      <hardwareInterface>hardware_interface/PositionJointInterface</hardwareInterface>
-    </joint>
-  </transmission>
-  <xacro:macro name="mimic_joint_plugin_gazebo" params="name_prefix parent_joint mimic_joint has_pid:=false multiplier:=1.0 offset:=0 sensitiveness:=0.0 max_effort:=1.0 robot_namespace:=''">
-    <gazebo>
-      <plugin name="${name_prefix}mimic_joint_plugin" filename="libroboticsgroup_gazebo_mimic_joint_plugin.so">
-        <joint>${parent_joint}</joint>
-        <mimicJoint>${mimic_joint}</mimicJoint>
-        <xacro:if value="${has_pid}">                     <!-- if set to true, PID parameters from "/gazebo_ros_control/pid_gains/${mimic_joint}" are loaded -->
-          <hasPID />
-        </xacro:if>
-        <multiplier>${multiplier}</multiplier>
-        <offset>${offset}</offset>
-        <sensitiveness>${sensitiveness}</sensitiveness>   <!-- if absolute difference between setpoint and process value is below this threshold, do nothing; 0.0 = disable [rad] -->
-        <maxEffort>${max_effort}</maxEffort>              <!-- only taken into account if has_pid:=true [Nm] -->
-        <xacro:unless value="${robot_namespace == ''}">
-          <robotNamespace>${robot_namespace}</robotNamespace>
-        </xacro:unless>
-      </plugin>
-    </gazebo>
-  </xacro:macro>
-  <xacro:mimic_joint_plugin_gazebo name_prefix="joint4"
-    parent_joint="joint2" mimic_joint="joint4"
-    has_pid="false" multiplier="1.0" max_effort="20.0"
-    robot_namespace="/$(arg robot_name)"/>
-  <xacro:mimic_joint_plugin_gazebo name_prefix="joint6"
-    parent_joint="joint5" mimic_joint="joint6"
-    has_pid="false" multiplier="1.0" max_effort="100.0"
-    robot_namespace="/$(arg robot_name)"/>
+      <hardwareInterface>hardware_interface/EffortJointInterface</hardwareInterface>
+    </joint>
+  </transmission>
+  <transmission name="tran6">
+    <type>transmission_interface/SimpleTransmission</type>
+    <actuator name="motor6">
+      <mechanicalReduction>1</mechanicalReduction>
+    </actuator>
+    <joint name="joint6">
+      <hardwareInterface>hardware_interface/EffortJointInterface</hardwareInterface>
+    </joint>
+  </transmission>
 </robot>

Commit message: Mess around with docker - got it working for gpu acceleration

File: catkin_ws/src/inserter_detector/simulation/inserter/inserter2.xacro (robot description, xacro)
@@ -27,4 +27,5 @@
       <!-- <robotNamespace>$(arg robot_name)</robotNamespace> -->
       <robotSimType>gazebo_ros_control/DefaultRobotHWSim</robotSimType>
+      <legacyModeNS>true</legacyModeNS>
     </plugin>
   </gazebo>
@@ -54,5 +55,5 @@
   </link>
   <joint name="joint1" type="revolute">
-    <limit effort="1000.0" lower="${-PI/2}" upper="${PI/2}" velocity="5"/>
+    <limit effort="1000.0" lower="${-PI}" upper="${PI}" velocity="5"/>
     <origin rpy="0 0 0" xyz="0 0 0"/> <!-- ${base_height + 0.01} -->
     <parent link="base_link"/>

File: catkin_ws/src/inserter_motion_planning/config/inserter.srdf.xacro (robot description, xacro)
@@ -14,10 +14,9 @@
         <joint name="joint2" />
         <joint name="joint3" />
-        <joint name="joint_arm_end" />
+        <link name="link4" />
     </group>
     <group name="$(arg robot_name)_hand">
-        <link name="link4" />
         <link name="link5" />
-        <!-- <link name="link6" /> -->
+        <link name="link6" />
     </group>
     <!--GROUP STATES: Purpose: Define a named state for a particular group, in terms of joint values. This is useful to define states like 'folded arms'-->
@@ -33,11 +32,9 @@
     </group_state>
     <!--END EFFECTOR: Purpose: Represent information about an end effector.-->
-    <end_effector name="$(arg robot_name)_hand" parent_link="link_arm_end" group="$(arg robot_name)_hand" parent_group="$(arg robot_name)_arm" />
+    <end_effector name="$(arg robot_name)_hand" parent_link="link4" group="$(arg robot_name)_hand" parent_group="$(arg robot_name)_arm" />
     <!--VIRTUAL JOINT: Purpose: this element defines a virtual joint between a robot link and an external frame of reference (considered fixed with respect to the robot)-->
     <!-- <virtual_joint name="virtual_joint" type="fixed" parent_frame="world" child_link="base_link" /> -->
     <!--PASSIVE JOINT: Purpose: this element is used to mark joints that are not actuated-->
-    <passive_joint name='joint_arm_end' />
     <passive_joint name="joint4" />
-    <passive_joint name="joint6" />
     <!--DISABLE COLLISIONS: By default it is assumed that any link of the robot could potentially come into collision with any other link in the robot. This tag disables collision checking between a specified pair of links. -->
     <disable_collisions link1="base_link" link2="link1" reason="Adjacent" />
